Commit message: load calibration from yaml file

File: urdf/alphasense.urdf.xacro (robot description, xacro)
@@ -1,6 +1,22 @@
 <?xml version="1.0"?>
+<!--
+Copyright 2022 University of Oxford
+Licensed under the Apache License, Version 2.0 (the "License");
+you may not use this file except in compliance with the License.
+You may obtain a copy of the License at
+    http://www.apache.org/licenses/LICENSE-2.0
+Unless required by applicable law or agreed to in writing, software
+distributed under the License is distributed on an "AS IS" BASIS,
+WITHOUT WARRANTIES OR CONDITIONS OF ANY KIND, either express or implied.
+See the License for the specific language governing permissions and
+limitations under the License.
+-->
 <robot name="alphasense" xmlns:xacro="http://www.ros.org/wiki/xacro">
-<xacro:macro name="alphasense" params="parent *origin name:=alphasense">
-  <joint name="${parent}_to_alphasense" type="fixed">
+<!-- YAML file containing the default values from CAD -->
+<xacro:property name="default_calib" value="$(find alphasense_description)/urdf/calibrations/default_calibration.yaml" />
+<xacro:macro name="alphasense" params="parent *origin name:=alphasense calib_file:=${default_calib}">
+<!-- load the YAML calibration file into a property -->
+<xacro:property name="calib" value="${load_yaml(calib_file)}"/>
+<joint name="${parent}_to_alphasense" type="fixed">
     <xacro:insert_block name="origin"/>
     <parent link="${parent}"/>
@@ -13,12 +29,12 @@
       </geometry>
     </visual>
-    <!-- TODO fix these inertial stuff -->
+    <!-- TODO check the inertia values -->
     <inertial>
-      <origin xzy="0 0 0" rpy="0 0 0"/>
+      <origin xyz="0 0 0" rpy="0 0 0"/>
       <mass value="0.5" />
       <inertia ixx="3.545e-4" ixy="6.051e-10" ixz="-3.736e-7" iyy="3.554e-4" iyz="-2.919e-9" izz="3.627e-4" />
     </inertial>
   </link>
-  <link name="imu_link">
+  <link name="${name}_imu">
     <visual>
       <geometry>
@@ -31,7 +47,7 @@
   </link>
   <joint name="imu_joint" type="fixed">
-    <origin xyz="6e-3 -8.55e-3 17.4e-3" rpy="${pi} 0 0"/>
+    <origin xyz="6.0e-3 -8.55e-3 17.4e-3" rpy="${pi} 0 0"/>
     <parent link="alphasense_mount" />
-    <child link="imu_link" />
+    <child link="${name}_imu" />
   </joint>
   <link name="cam_front_left">
@@ -75,27 +91,72 @@
     </visual>
   </link>
+  <link name="cam_top">
+    <visual>
+      <geometry>
+        <box size="1e-3 1e-3 1e-3" />
+      </geometry>
+      <material name="black">
+        <color rgba="0 0 0 1" />
+      </material>
+    </visual>
+  </link>
   <!-- front right camera which is cam0 in alphasense driver -->
-  <joint name="front_right_cam_joint" type="fixed">
-    <origin xyz="0.0438 0.0485 -0.0109" rpy="1.5708 0.0043 1.5675 "/>
-    <parent link="imu_link" />
+  <joint name="imu_to_cam_front_right_joint" type="fixed">
+    <!--origin xyz="0.0438 0.0485 -0.0109" rpy="1.5708 0.0043 1.5675 "/-->
+    <origin xyz="${calib['imu_to_cam0']['x']}
+                 ${calib['imu_to_cam0']['y']}
+                 ${calib['imu_to_cam0']['z']}"
+            rpy="${calib['imu_to_cam0']['roll']}
+                 ${calib['imu_to_cam0']['pitch']}
+                 ${calib['imu_to_cam0']['yaw']}"/>
+    <parent link="${name}_imu" />
     <child link="cam_front_right" />
   </joint>
   <!-- front left camera which is cam1 in alphasense driver -->
-  <joint name="front_left_cam_joint" type="fixed">
-    <origin xyz="0.0437 -0.0611 -0.0115" rpy=" 1.5715 -0.0042 1.5712 "/>
-    <parent link="imu_link" />
+  <joint name="imu_to_cam_front_left_joint" type="fixed">
+    <!--origin xyz="0.0437 -0.0611 -0.0115" rpy=" 1.5715 -0.0042 1.5712 "/-->
+    <origin xyz="${calib['imu_to_cam1']['x']}
+                 ${calib['imu_to_cam1']['y']}
+                 ${calib['imu_to_cam1']['z']}"
+            rpy="${calib['imu_to_cam1']['roll']}
+                 ${calib['imu_to_cam1']['pitch']}
+                 ${calib['imu_to_cam1']['yaw']}"/>
+    <parent link="${name}_imu" />
     <child link="cam_front_left" />
   </joint>
   <!-- top camera which is cam2 in alphasense driver, haven't calibrated yet -->
+  <joint name="imu_to_cam_top_joint" type="fixed">
+    <!--origin xyz="-0.00789 -0.07720 -0.01356" rpy="1.5733 0.00443 -0.0052"/-->
+    <origin xyz="${calib['imu_to_cam2']['x']}
+                 ${calib['imu_to_cam2']['y']}
+                 ${calib['imu_to_cam2']['z']}"
+            rpy="${calib['imu_to_cam2']['roll']}
+                 ${calib['imu_to_cam2']['pitch']}
+                 ${calib['imu_to_cam2']['yaw']}"/>
+    <parent link="${name}_imu" />
+    <child link="cam_top" />
+  </joint>
   <!-- side right camera which is cam3 in alphasense driver -->
-  <joint name="side_right_cam_joint" type="fixed">
-    <origin xyz="-0.006 0.062 -0.0105" rpy="1.5691 -0.0061 3.1334"/>
-    <parent link="imu_link" />
+  <joint name="imu_to_cam_side_right_joint" type="fixed">
+    <!--origin xyz="-0.006 0.062 -0.0105" rpy="1.5691 -0.0061 3.1334"/-->
+    <origin xyz="${calib['imu_to_cam3']['x']}
+                 ${calib['imu_to_cam3']['y']}
+                 ${calib['imu_to_cam3']['z']}"
+            rpy="${calib['imu_to_cam3']['roll']}
+                 ${calib['imu_to_cam3']['pitch']}
+                 ${calib['imu_to_cam3']['yaw']}"/>
+    <parent link="${name}_imu" />
     <child link="cam_side_right" />
   </joint>
   <!-- side left camera which is cam4 in alphasense driver -->
-  <joint name="side_left_cam_joint" type="fixed">
-    <origin xyz="-0.00789 -0.07720 -0.01356" rpy="1.5733 0.00443 -0.0052"/>
-    <parent link="imu_link" />
+  <joint name="imu_to_cam_side_left_joint" type="fixed">
+    <!--origin xyz="-0.00789 -0.07720 -0.01356" rpy="1.5733 0.00443 -0.0052"/-->
+    <origin xyz="${calib['imu_to_cam4']['x']}
+                 ${calib['imu_to_cam4']['y']}
+                 ${calib['imu_to_cam4']['z']}"
+            rpy="${calib['imu_to_cam4']['roll']}
+                 ${calib['imu_to_cam4']['pitch']}
+                 ${calib['imu_to_cam4']['yaw']}"/>
+    <parent link="${name}_imu" />
     <child link="cam_side_left" />
   </joint>

File: urdf/alphasense_standalone.urdf.xacro (robot description, xacro)
@@ -1,3 +1,15 @@
 <?xml version="1.0" ?>
+<!--
+Copyright 2022 University of Oxford
+Licensed under the Apache License, Version 2.0 (the "License");
+you may not use this file except in compliance with the License.
+You may obtain a copy of the License at
+    http://www.apache.org/licenses/LICENSE-2.0
+Unless required by applicable law or agreed to in writing, software
+distributed under the License is distributed on an "AS IS" BASIS,
+WITHOUT WARRANTIES OR CONDITIONS OF ANY KIND, either express or implied.
+See the License for the specific language governing permissions and
+limitations under the License.
+-->
 <robot name="alphasense_standalone" xmlns:xacro="http://www.ros.org/wiki/xacro">
   <xacro:include filename="$(find alphasense_description)/urdf/alphasense.urdf.xacro" />

Commit message: changes to support ros2

File: urdf/alphasense.urdf.xacro (robot description, xacro)
@@ -26,5 +26,5 @@
     <visual>
       <geometry>
-        <mesh filename="package://alphasense_description/urdf/meshes/alphasense_simplified.dae" />
+        <mesh filename="$(find alphasense_description)/urdf/meshes/alphasense_simplified.dae" />
       </geometry>
     </visual>

Commit message: allow rviz loading

File: urdf/alphasense.urdf.xacro (robot description, xacro)
@@ -17,5 +17,5 @@
 <xacro:macro name="alphasense" params="parent *origin name:=alphasense calib_file:=${default_calib}">
 <!-- load the YAML calibration file into a property -->
-<xacro:property name="calib" value="${load_yaml(calib_file)}"/>
+<xacro:property name="calib" value="${xacro.load_yaml(calib_file)}"/>
 <joint name="${parent}_to_alphasense" type="fixed">
     <xacro:insert_block name="origin"/>
@@ -26,5 +26,5 @@
     <visual>
       <geometry>
-        <mesh filename="$(find alphasense_description)/urdf/meshes/alphasense_simplified.dae" />
+        <mesh filename="package://alphasense_description/urdf/meshes/alphasense_simplified.dae" />
       </geometry>
     </visual>

File: urdf/alphasense_standalone.urdf (robot description, URDF)
Before this commit: robot alphasense_standalone, 7 links, 6 joints
Links:
- link alphasense_mount: geometry 
